File: Prototype5/schematic/Prototype5.sch (KiCad schematic (older format))
At the start: 18 parts, among them J1 Conn_AVR_UPDI, SW1 TSD1265, U1 ATmega4809-P, U2 HM628128DLP-5, U3 HD63C09E, U5 CD74HCT30, U6 CD74HCT688

Commit message: [CyborgHD6309E] Prorotype5 debugger
Parts:
- removed U5: CD74HCT30, Package_DIP:DIP-14_W7.62mm, symbol 0-LocalLibrary:74HC30
- added C4: 18p, symbol Device:C_Small
- added R1, R4: 18, symbol Device:R_Small
- added RN1: 100k, Resistor_THT:R_Array_SIP9, symbol Device:R_Network08
- added SW2: SW_DIP_x08, Package_DIP:DIP-16_W7.62mm, symbol Switch:SW_DIP_x08
- C5: value 0.1u -> 18p; footprint Capacitor_THT:C_Disc_D3.4mm_W2.1mm_P2.50mm -> (none)
Connections:
- net A0: now also U2.12 (A0); no longer U2.26 (A9)
- net A1: now also U2.11 (A1); no longer U2.25 (A11)
- net A10: now also U2.23 (A10), U6.6 (A2); no longer U2.10 (A2)
- net A11: now also U2.25 (A11), U6.8 (A3); no longer U2.11 (A1)
- net A12: now also U2.4 (A12), U6.11 (A4); no longer U2.12 (A0)
- net A13: now also U2.28 (A13), U6.13 (A5); no longer U2.27 (A8)
- net A14: now also U2.3 (A14), U6.15 (A6); no longer U2.28 (A13)
- net A15: now also U6.17 (A7)
- net A2: now also U2.10 (A2); no longer U2.23 (A10)
- net A3: now also U2.9 (A3); no longer U2.3 (A14), U6.17 (A7)
- net A4: now also U2.8 (A4); no longer U2.4 (A12), U6.15 (A6)
- net A5: now also U2.7 (A5); no longer U2.5 (A7), U6.13 (A5)
- net A6: no longer U6.11 (A4)
- net A7: now also U2.5 (A7); no longer U2.7 (A5), U6.8 (A3)
- net A8: now also U2.27 (A8), U6.2 (A0); no longer U2.8 (A4)
- net A9: now also U2.26 (A9), U6.4 (A1); no longer U2.9 (A3)
- net D0: now also U2.13 (Q0); no longer U2.21 (Q7)
- net D1: now also U2.14 (Q1); no longer U2.20 (Q6)
- net D2: now also U2.15 (Q2); no longer U2.19 (Q5)
- net D3: now also U2.17 (Q3); no longer U2.18 (Q4)
- net D4: now also U2.18 (Q4); no longer U2.17 (Q3)
- net D5: now also U2.19 (Q5); no longer U2.13 (Q0)
- net D6: now also U2.20 (Q6); no longer U2.14 (Q1)
- net D7: now also U2.21 (Q7); no longer U2.15 (Q2)
- net E_CLK: now also U1.25 (PF2), R1.1; no longer U1.26 (PF3), U3.35 (Q)
- net GND: now also U6.1 (~E~), C4.1, SW2.10, SW2.11, SW2.12, SW2.13, SW2.14, SW2.15, SW2.16, SW2.9; no longer U6.14 (B5), U6.16 (B6), U6.18 (B7), U6.2 (A0), U6.3 (B0), U6.4 (A1), U6.5 (B1), U6.6 (A2), U6.7 (B2)
- net Q_CLK: now also U1.3 (PC2/SDA), R4.1; no longer U1.4 (PC3/SCL), U3.34 (E)
- net VCC: now also RN1.1 (common); no longer C5.1, U6.12 (B4), U6.9 (B3)
- net ~IOR~: now also U1.26 (PF3); no longer U1.25 (PF2)
- net ~RAM_E~: now also U1.4 (PC3/SCL); no longer U1.3 (PC2/SDA)
- new net: C4.2, C5.1, R1.2, R4.2, U3.34 (E), U3.35 (Q)
- new net: RN1.6 (R5), SW2.5, U6.12 (B4)
- new net: RN1.7 (R6), SW2.6, U6.14 (B5)
- new net: RN1.8 (R7), SW2.7, U6.16 (B6)
- new net: RN1.9 (R8), SW2.8, U6.18 (B7)
- new net: RN1.2 (R1), SW2.1, U6.3 (B0)
- new net: RN1.3 (R2), SW2.2, U6.5 (B1)
- new net: RN1.4 (R3), SW2.3, U6.7 (B2)
- new net: RN1.5 (R4), SW2.4, U6.9 (B3)
Other:
- moved on the sheet: C6, U6
