File: Prototype3/schematic/Prototype3.kicad_pcb (KiCad board)
At the start: 2 copper layers, 95 x 72 mm, 29 parts, among them J1 Conn_USB_Serial, J2 Conn_AVR_ISP, J3 Conn_Micro_SD, J4 Conn_AVR_ISP, SW1 USR_SW, U1 ATmega1284P-PU, U2 HM628128DLP-5, U3 HD63C09E, U4 ATmega328P-PU, Y1 20MHz, Y2 20MHz

Commit message: Migrate to KiCad 6.0
Connections:
- net /~ACK~ renamed /~{ACK}
- net /~DBG_RST~ renamed /~{DBG_RST}
- net /~HALT~ renamed /~{HALT}
- net /~INT~ renamed /~{INT}
- net /~IRQ renamed /~{IRQ}
- net /~NMI~ renamed /~{NMI}
- net /~RAM_E~ renamed /~{RAM_E}
- net /~RESET~ renamed /~{RESET}
- net /~SD_CS~ renamed /~{SD_CS}
- net /~STEP~ renamed /~{STEP}
- net /~USR_SW~ renamed /~{USR_SW}
Other:
- net class Default removed
