File: Prototype3/schematic/Prototype3.kicad_sch (KiCad schematic)
At the start: 25 parts, among them J1 Conn_USB_Serial, J2 Conn_AVR_ISP, J3 Conn_Micro_SD, J4 Conn_AVR_ISP, SW1 USR_SW, U1 ATmega1284P-PU, U2 HM628128DLP-5, U3 HD63C09E, U4 ATmega328P-PU, Y1 20MHz, Y2 20MHz

Commit message: Satisfy Electrical Rules Checker
Parts:
- removed J1: Conn_USB_Serial, Connector_PinSocket_2.54mm:PinSocket_1x06_P2.54mm_Vertical, symbol Prototype3-rescue:Conn_USB_Serial-0-LocalLibrary
- removed J3: Conn_Micro_SD, Connector_PinSocket_2.54mm:PinSocket_1x07_P2.54mm_Vertical, symbol Prototype3-rescue:Conn_Micro_SD-0-LocalLibrary
- added B1: USB_Serial, 0-LocalLibrary:GY232V2, symbol 0-LocalLibrary:USB_Serial
- added B2: Micro_SD, 0-LocalLibrary:uSD_CARD, symbol 0-LocalLibrary:Micro_SD
Connections:
- net DBG_RX: now also B1.4 (TXD)
- net DBG_TX: now also B1.5 (RXD)
- net GND: now also B1.1 (GND), B1.2 (~{CTS}), B2.7 (GND)
- net SD_DI: now also B2.3 (DI)
- net SD_DO: now also B2.5 (DO)
- net SD_SCK: now also B2.4 (SCK)
- net VCC: now also B1.3 (5V0), B2.1 (VCC)
- net ~{SD_CS}: now also B2.2 (~{CS})
- net at C2.1: now also B1.6 (~{DTR})
Changed lines of the file:
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@@
   (junction (at 81.28 105.41) (diameter 0) (color 0 0 0 0)
   )
+  (junction (at 191.77 102.87) (diameter 0) (color 0 0 0 0)
+  )
+  (junction (at 44.45 107.95) (diameter 0) (color 0 0 0 0)
+  )
+  (junction (at 215.9 90.17) (diameter 0) (color 0 0 0 0)
+  )
+  (junction (at 252.73 52.07) (diameter 0) (color 0 0 0 0)
+  )
   (junction (at 64.77 149.86) (diameter 0) (color 0 0 0 0)
-  )
-  (junction (at 191.77 102.87) (diameter 0) (color 0 0 0 0)
-  )
-  (junction (at 44.45 107.95) (diameter 0) (color 0 0 0 0)
-  )
-  (junction (at 215.9 90.17) (diameter 0) (color 0 0 0 0)
-  )
-  (junction (at 252.73 52.07) (diameter 0) (color 0 0 0 0)
   )
   (junction (at 138.43 34.29) (diameter 0) (color 0 0 0 0)
@@
     (stroke (width 0) (type default) (color 0 0 0 0))
   )
+  (wire (pts (xy 64.77 149.86) (xy 66.04 149.86))
+    (stroke (width 0) (type default) (color 0 0 0 0))
+  )
   (wire (pts (xy 39.37 90.17) (xy 46.99 90.17))
     (stroke (width 0) (type default) (color 0 0 0 0))
@@
     (stroke (width 0) (type default) (color 0 0 0 0))
   )
-  (wire (pts (xy 64.77 149.86) (xy 63.5 149.86))
-    (stroke (width 0) (type default) (color 0 0 0 0))
-  )
   (wire (pts (xy 105.41 69.85) (xy 109.22 69.85))
     (stroke (width 0) (type default) (color 0 0 0 0))
@@
     (stroke (width 0) (type default) (color 0 0 0 0))
   )
-  (wire (pts (xy 66.04 149.86) (xy 64.77 149.86))
+  (wire (pts (xy 63.5 149.86) (xy 64.77 149.86))
     (stroke (width 0) (type default) (color 0 0 0 0))
   )
@@
     (effects (font (size 1.27 1.27)) (justify right bottom))
   )
+  (label "D[0..7]" (at 54.61 34.29 0)
+    (effects (font (size 1.27 1.27)) (justify left bottom))
+  )
   (label "BS" (at 77.47 69.85 0)
     (effects (font (size 1.27 1.27)) (justify left bottom))
@@
   )
   (label "E_CLK" (at 246.38 80.01 0)
+    (effects (font (size 1.27 1.27)) (justify left bottom))
+  )
+  (label "A[0..15]" (at 54.61 36.83 0)
     (effects (font (size 1.27 1.27)) (justify left bottom))
   )
@@
     )
     (property "Datasheet" "" (id 3) (at 134.62 97.79 0)
-      (effects (font (size 1.27 1.27)) hide)
-    )
-    (pin "1")
-  )
-  (symbol (lib_id "power:VCC") (at -1352.55 -1136.65 0) (unit 1)
-    (in_bom yes) (on_board yes)
-    (property "Reference" "#PWR01" (id 0) (at -1352.55 -1132.84 0)
-      (effects (font (size 1.27 1.27)) hide)
-    )
-    (property "Value" "VCC" (id 1) (at -1352.1182 -1141.0442 0))
-    (property "Footprint" "" (id 2) (at -1352.55 -1136.65 0)
-      (effects (font (size 1.27 1.27)) hide)
-    )
-    (property "Datasheet" "" (id 3) (at -1352.55 -1136.65 0)
       (effects (font (size 1.27 1.27)) hide)
     )
@@
     (pin "2")
   )
-  (symbol (lib_id "power:GND") (at -15.24 -91.44 0) (unit 1)
-    (in_bom yes) (on_board yes)
-    (property "Reference" "#PWR02" (id 0) (at -15.24 -85.09 0)
-      (effects (font (size 1.27 1.27)) hide)
-    )
-    (property "Value" "GND" (id 1) (at -15.113 -87.0458 0))
-    (property "Footprint" "" (id 2) (at -15.24 -91.44 0)
-      (effects (font (size 1.27 1.27)) hide)
-    )
-    (property "Datasheet" "" (id 3) (at -15.24 -91.44 0)
-      (effects (font (size 1.27 1.27)) hide)
-    )
-    (pin "1")
-  )
   (symbol (lib_id "power:GND") (at 148.59 153.67 0) (unit 1)
     (in_bom yes) (on_board yes)
@@
     (pin "1")
     (pin "2")
-  )
-  (symbol (lib_id "Prototype3-rescue:Conn_Micro_SD-0-LocalLibrary") (at 153.67 146.05 0) (unit 1)
-    (in_bom yes) (on_board yes)
-    (property "Reference" "J3" (id 0) (at 153.67 134.62 0)
-      (effects (font (size 1.27 1.27)) (justify left))
-    )
-    (property "Value" "Conn_Micro_SD" (id 1) (at 151.13 157.48 0)
-      (effects (font (size 1.27 1.27)) (justify left))
-    )
-    (property "Footprint" "Connector_PinSocket_2.54mm:PinSocket_1x07_P2.54mm_Vertical" (id 2) (at 153.67 146.05 0)
-      (effects (font (size 1.27 1.27)) hide)
-    )
-    (property "Datasheet" "~" (id 3) (at 153.67 146.05 0)
-      (effects (font (size 1.27 1.27)) hide)
-    )
-    (pin "1")
-    (pin "2")
-    (pin "3")
-    (pin "4")
-    (pin "5")
-    (pin "6")
-    (pin "7")
-  )
-  (symbol (lib_id "Prototype3-rescue:Conn_USB_Serial-0-LocalLibrary") (at 69.85 142.24 0) (unit 1)
-    (in_bom yes) (on_board yes)
-    (property "Reference" "J1" (id 0) (at 69.85 133.35 0)
-      (effects (font (size 1.27 1.27)) (justify left))
-    )
-    (property "Value" "Conn_USB_Serial" (id 1) (at 66.04 157.48 0)
-      (effects (font (size 1.27 1.27)) (justify left))
-    )
-    (property "Footprint" "Connector_PinSocket_2.54mm:PinSocket_1x06_P2.54mm_Vertical" (id 2) (at 69.85 142.24 0)
-      (effects (font (size 1.27 1.27)) hide)
-    )
-    (property "Datasheet" "~" (id 3) (at 69.85 142.24 0)
-      (effects (font (size 1.27 1.27)) hide)
-    )
-    (pin "1")
-    (pin "2")
-    (pin "3")
-    (pin "4")
-    (pin "5")
-    (pin "6")
   )
   (symbol (lib_id "power:VCC") (at 55.88 129.54 0) (unit 1)
@@
     (pin "1")
   )
+  (symbol (lib_id "0-LocalLibrary:USB_Serial") (at 69.85 142.24 0) (unit 1)
+    (in_bom yes) (on_board yes)
+    (property "Reference" "B1" (id 0) (at 68.58 133.35 0)
+      (effects (font (size 1.27 1.27)) (justify left))
+    )
+    (property "Value" "USB_Serial" (id 1) (at 71.12 153.67 0)
+      (effects (font (size 1.27 1.27)) (justify left))
+    )
+    (property "Footprint" "0-LocalLibrary:GY232V2" (id 2) (at 69.85 153.67 0)
+      (effects (font (size 1.27 1.27)) hide)
+    )
+    (property "Datasheet" "~" (id 3) (at 69.85 142.24 0)
+      (effects (font (size 1.27 1.27)) hide)
+    )
+    (pin "1")
+    (pin "2")
+    (pin "3")
+    (pin "4")
+    (pin "5")
+    (pin "6")
+  )
+  (symbol (lib_id "0-LocalLibrary:Micro_SD") (at 153.67 146.05 0) (unit 1)
+    (in_bom yes) (on_board yes)
+    (property "Reference" "B2" (id 0) (at 152.4 134.62 0)
+      (effects (font (size 1.27 1.27)) (justify left))
+    )
+    (property "Value" "Micro_SD" (id 1) (at 153.67 157.48 0)
+      (effects (font (size 1.27 1.27)) (justify left))
+    )
+    (property "Footprint" "0-LocalLibrary:uSD_CARD" (id 2) (at 153.67 146.05 0)
+      (effects (font (size 1.27 1.27)) hide)
+    )
+    (property "Datasheet" "~" (id 3) (at 153.67 146.05 0)
+      (effects (font (size 1.27 1.27)) hide)
+    )
+    (pin "1")
+    (pin "2")
+    (pin "3")
+    (pin "4")
+    (pin "5")
+    (pin "6")
+    (pin "7")
+  )
   (sheet_instances
     (path "/" (page "1"))
   )
   (symbol_instances
-    (path "/00000000-0000-0000-0000-00005cde46a4"
-      (reference "#PWR01") (unit 1) (value "VCC") (footprint "")
-    )
-    (path "/00000000-0000-0000-0000-00005d0883ef"
-      (reference "#PWR02") (unit 1) (value "GND") (footprint "")
-    )
     (path "/00000000-0000-0000-0000-00005ce5efde"
       (reference "#PWR03") (unit 1) (value "VCC") (footprint "")
@@
       (reference "#PWR026") (unit 1) (value "GND") (footprint "")
     )
+    (path "/d3959c2e-abdb-43d9-80a9-65b67b43f57c"
+      (reference "B1") (unit 1) (value "USB_Serial") (footprint "0-LocalLibrary:GY232V2")
+    )
+    (path "/fe2b97af-f6e6-47c9-b8c8-b73522c97b29"
+      (reference "B2") (unit 1) (value "Micro_SD") (footprint "0-LocalLibrary:uSD_CARD")
+    )
     (path "/00000000-0000-0000-0000-00005d080349"
       (reference "C1") (unit 1) (value "0.1u") (footprint "Capacitor_SMD:C_0603_1608Metric")
@@
       (reference "D1") (unit 1) (value "USR_LED") (footprint "LED_THT:LED_D3.0mm")
     )
-    (path "/00000000-0000-0000-0000-00005d0b116c"
-      (reference "J1") (unit 1) (value "Conn_USB_Serial") (footprint "Connector_PinSocket_2.54mm:PinSocket_1x06_P2.54mm_Vertical")
-    )
     (path "/00000000-0000-0000-0000-00005d3e967f"
       (reference "J2") (unit 1) (value "Conn_AVR_ISP") (footprint "Connector_PinSocket_2.54mm:PinSocket_1x06_P2.54mm_Vertical")
     )
-    (path "/00000000-0000-0000-0000-00005d0a3a84"
-      (reference "J3") (unit 1) (value "Conn_Micro_SD") (footprint "Connector_PinSocket_2.54mm:PinSocket_1x07_P2.54mm_Vertical")
-    )
     (path "/00000000-0000-0000-0000-00005d32154a"
