File: Prototype4/schematic/Prototype4.kicad_pcb (KiCad board)
At the start: 2 copper layers, 95 x 72 mm, 24 parts, among them J1 Conn_AVR_UPDI, SW1 TSD1265, U1 ATmega4809-P, U2 HM628128DLP-5, U3 HD63C09E, U4 ATtiny412-SS, U5 CD74HCT30, U6 CD74HCT688

Commit message: Migrate to KiCad 6.0
Connections:
- net /~ACK~ renamed /~{ACK}
- net /~DBG_RESET~ renamed /~{DBG_RESET}
- net /~HALT~ renamed /~{HALT}
- net /~INT~ renamed /~{INT}
- net /~IRQ~ renamed /~{IRQ}
- net /~NMI~ renamed /~{NMI}
- net /~RAM_E~ renamed /~{RAM_E}
- net /~RESET~ renamed /~{RESET}
- net /~SD_CS~ renamed /~{SD_CS}
- net /~STEP~ renamed /~{STEP}
- net /~USR_SW~ renamed /~{USR_SW}
Other:
- net class Default removed
