File: Prototype4/schematic/Prototype4.kicad_sch (KiCad schematic)
At the start: 20 parts, among them J1 Conn_AVR_UPDI, SW1 TSD1265, U1 ATmega4809-P, U2 HM628128DLP-5, U3 HD63C09E, U4 ATtiny412-SS, U5 CD74HCT30, U6 CD74HCT688

Commit message: Satisfy Electrical Rules Checker
Changed lines of the file:
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@@
     (effects (font (size 1.27 1.27)) (justify right bottom))
+  )
+  (label "A[0..15]" (at 185.42 31.75 0)
+    (effects (font (size 1.27 1.27)) (justify left bottom))
   )
   (label "A5" (at 152.4 64.77 180)
@@
   (label "A9" (at 101.6 59.69 180)
     (effects (font (size 1.27 1.27)) (justify right bottom))
+  )
+  (label "D[0..7]" (at 156.21 29.21 0)
+    (effects (font (size 1.27 1.27)) (justify left bottom))
   )
   (label "A12" (at 201.93 57.15 180)
@@
     )
     (property "Datasheet" "" (id 3) (at 128.27 99.06 0)
-      (effects (font (size 1.27 1.27)) hide)
-    )
-    (pin "1")
-  )
-  (symbol (lib_id "power:VCC") (at -1352.55 -1136.65 0) (unit 1)
-    (in_bom yes) (on_board yes)
-    (property "Reference" "#PWR01" (id 0) (at -1352.55 -1132.84 0)
-      (effects (font (size 1.27 1.27)) hide)
-    )
-    (property "Value" "VCC" (id 1) (at -1352.1182 -1141.0442 0))
-    (property "Footprint" "" (id 2) (at -1352.55 -1136.65 0)
-      (effects (font (size 1.27 1.27)) hide)
-    )
-    (property "Datasheet" "" (id 3) (at -1352.55 -1136.65 0)
       (effects (font (size 1.27 1.27)) hide)
     )
@@
   )
   (symbol_instances
-    (path "/00000000-0000-0000-0000-00005cde46a4"
-      (reference "#PWR01") (unit 1) (value "VCC") (footprint "")
-    )
     (path "/00000000-0000-0000-0000-00005ce5efde"
       (reference "#PWR02") (unit 1) (value "VCC") (footprint "")
