File: schematic/Prototype5.kicad_pcb (KiCad board)
At the start: 2 copper layers, 95 x 72 mm, 22 parts, among them J1 Conn_AVR_UPDI, SW1 TSD1265, SW2 SW_DIP_x08, U1 ATmega4809-P, U2 HM628128DLP-5, U3 HD63C09E, U6 CD74HCT688

Commit message: Migrate to KiCad 6.0
Connections:
- net /~DBG_RESET~ renamed /~{DBG_RESET}
- net /~HALT~ renamed /~{HALT}
- net /~IOR~ renamed /~{IOR}
- net /~IRQ~ renamed /~{IRQ}
- net /~NMI~ renamed /~{NMI}
- net /~RAM_E~ renamed /~{RAM_E}
- net /~RESET~ renamed /~{RESET}
- net /~SD_CS~ renamed /~{SD_CS}
- net /~USR_SW~ renamed /~{USR_SW}
Other:
- net class Default removed
