File: schematic/Prototype5.kicad_sch (KiCad schematic)
At the start: 22 parts, among them J1 Conn_AVR_UPDI, SW1 TSD1265, SW2 SW_DIP_x08, U1 ATmega4809-P, U2 HM628128DLP-5, U3 HD63C09E, U6 CD74HCT688

Commit message: Satisfy Electrical Rules Checker
Changed lines of the file:
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@@
+    (effects (font (size 1.27 1.27)) (justify left bottom))
+  )
+  (label "A[0..15]" (at 156.21 31.75 0)
     (effects (font (size 1.27 1.27)) (justify left bottom))
   )
@@
   )
   (label "~{DBG_RESET}" (at 80.01 91.44 0)
+    (effects (font (size 1.27 1.27)) (justify left bottom))
+  )
+  (label "D[0..7]" (at 156.21 29.21 0)
     (effects (font (size 1.27 1.27)) (justify left bottom))
   )
@@
     )
     (property "Datasheet" "" (id 3) (at 128.27 99.06 0)
-      (effects (font (size 1.27 1.27)) hide)
-    )
-    (pin "1")
-  )
-  (symbol (lib_id "power:VCC") (at -1352.55 -1136.65 0) (unit 1)
-    (in_bom yes) (on_board yes)
-    (property "Reference" "#PWR01" (id 0) (at -1352.55 -1132.84 0)
-      (effects (font (size 1.27 1.27)) hide)
-    )
-    (property "Value" "VCC" (id 1) (at -1352.1182 -1141.0442 0))
-    (property "Footprint" "" (id 2) (at -1352.55 -1136.65 0)
-      (effects (font (size 1.27 1.27)) hide)
-    )
-    (property "Datasheet" "" (id 3) (at -1352.55 -1136.65 0)
       (effects (font (size 1.27 1.27)) hide)
     )
@@
   )
   (symbol_instances
-    (path "/00000000-0000-0000-0000-00005cde46a4"
-      (reference "#PWR01") (unit 1) (value "VCC") (footprint "")
-    )
     (path "/00000000-0000-0000-0000-00005ce5efde"
       (reference "#PWR02") (unit 1) (value "VCC") (footprint "")
